File: HARDWARE/TER_PEDAL/MICRO.kicad_sch (KiCad schematic)
At the start: 22 parts, among them J1 DEBUG, SW1 RST, U1 STM32F103C8Tx, Y1 8mHz

Commit message: Rearranged board
Parts:
- Y1: footprint Crystal:Crystal_HC52-6mm_Vertical -> Crystal:Crystal_SMD_5032-2Pin_5.0x3.2mm
Changed lines of the file:
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@@
       (effects (font (size 1.27 1.27)))
     )
-    (property "Footprint" "Crystal:Crystal_HC52-6mm_Vertical" (at 31.75 157.48 0)
+    (property "Footprint" "Crystal:Crystal_SMD_5032-2Pin_5.0x3.2mm" (at 31.75 157.48 0)
       (effects (font (size 1.27 1.27)) hide)
     )

Commit message: Finished Routing for redisign
Connections:
- net APPS_1_ADC: now also U1.17 (PA7); no longer U1.16 (PA6)
- net APPS_2_ADC: now also U1.18 (PB0); no longer U1.17 (PA7)
- net STEER_ADC: now also U1.16 (PA6); no longer U1.18 (PB0)
Changed lines of the file:
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@@
     (effects (font (size 1.27 1.27)) (justify left))
   )
-  (hierarchical_label "APPS_1_ADC" (shape input) (at 161.29 66.04 0) (fields_autoplaced)
+  (hierarchical_label "APPS_2_ADC" (shape input) (at 118.11 78.74 180) (fields_autoplaced)
+    (effects (font (size 1.27 1.27)) (justify right))
+  )
+  (hierarchical_label "APPS_1_ADC" (shape input) (at 161.29 68.58 0) (fields_autoplaced)
     (effects (font (size 1.27 1.27)) (justify left))
   )
@@
     (effects (font (size 1.27 1.27)) (justify right))
   )
-  (hierarchical_label "STEER_ADC" (shape input) (at 118.11 78.74 180) (fields_autoplaced)
-    (effects (font (size 1.27 1.27)) (justify right))
-  )
-  (hierarchical_label "APPS_2_ADC" (shape input) (at 161.29 68.58 0) (fields_autoplaced)
+  (hierarchical_label "STEER_ADC" (shape input) (at 161.29 66.04 0) (fields_autoplaced)
     (effects (font (size 1.27 1.27)) (justify left))
   )

Commit message: Quick Fix on the debug conector Bus where it was not connected to 3.3V + Labels
Parts:
- FB1: footprint Inductor_SMD:L_0402_1005Metric -> Inductor_SMD:L_0805_2012Metric
Connections:
- net +3V3 is gone; now on net +3.3V: J1.4 (Pin_4)
Changed lines of the file:
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@@
+    )
+  )
+  (symbol (lib_id "power:+3.3V") (at 256.54 41.91 180) (unit 1)
+    (in_bom yes) (on_board yes) (dnp no) (fields_autoplaced)
+    (property "Reference" "#PWR02" (at 256.54 38.1 0)
+      (effects (font (size 1.27 1.27)) hide)
+    )
+    (property "Value" "+3.3V" (at 256.54 46.99 0)
+      (effects (font (size 1.27 1.27)))
+    )
+    (property "Footprint" "" (at 256.54 41.91 0)
+      (effects (font (size 1.27 1.27)) hide)
+    )
+    (property "Datasheet" "" (at 256.54 41.91 0)
+      (effects (font (size 1.27 1.27)) hide)
+    )
+    (pin "1")
+    (instances
+      (project "TER_PEDAL"
+        (path "/73ede3a3-6344-40fe-9207-10ff50d388ba"
+          (reference "#PWR02") (unit 1)
+        )
+        (path "/73ede3a3-6344-40fe-9207-10ff50d388ba/7632a94a-0691-4527-83e2-6d814eae7e64"
+          (reference "#PWR033") (unit 1)
+        )
+      )
     )
   )
@@
     )
   )
-  (symbol (lib_name "+3.3V_1") (lib_id "power:+3.3V") (at 256.54 41.91 180) (unit 1)
-    (in_bom yes) (on_board yes) (dnp no) (fields_autoplaced)
-    (property "Reference" "#PWR033" (at 256.54 38.1 0)
-      (effects (font (size 1.27 1.27)) hide)
-    )
-    (property "Value" "+3.3V" (at 256.54 46.99 0)
-      (effects (font (size 1.27 1.27)))
-    )
-    (property "Footprint" "" (at 256.54 41.91 0)
-      (effects (font (size 1.27 1.27)) hide)
-    )
-    (property "Datasheet" "" (at 256.54 41.91 0)
-      (effects (font (size 1.27 1.27)) hide)
-    )
-    (pin "1")
-    (instances
-      (project "TER_PEDAL"
-        (path "/73ede3a3-6344-40fe-9207-10ff50d388ba/7632a94a-0691-4527-83e2-6d814eae7e64"
-          (reference "#PWR033") (unit 1)
-        )
-      )
-    )
-  )
   (symbol (lib_id "power:GND") (at 15.24 30.48 0) (unit 1)
     (in_bom yes) (on_board yes) (dnp no) (fields_autoplaced)
@@
       (effects (font (size 1.27 1.27)))
     )
-    (property "Footprint" "Inductor_SMD:L_0402_1005Metric" (at 35.56 52.578 90)
-      (effects (font (size 1.27 1.27)) hide)
-    )
+    (property "Footprint" "Inductor_SMD:L_0805_2012Metric" (at 35.56 52.578 90)
+      (effects (font (size 1.27 1.27)) hide)
+    )

Commit message: Bumped Bugfix version and fixed unnecessary BOOT0 pin and rj45 placement
Parts:
- removed JP2: BOOT1, Connector_PinHeader_2.00mm:PinHeader_1x03_P2.00mm_Vertical, symbol Jumper:Jumper_3_Bridged12
- removed R5: 10k, Resistor_SMD:R_0603_1608Metric, symbol Device:R_Small
Connections:
- net BOOT1 is gone; now on net GND: U1.20 (PB2)
Changed lines of the file:
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@@
-    (stroke (width 0) (type default))
-  )
-  (wire (pts (xy 40.64 121.92) (xy 40.64 125.73))
     (stroke (width 0) (type default))
   )
@@
     (stroke (width 0) (type default))
   )
-  (wire (pts (xy 48.26 110.49) (xy 48.26 111.76))
-    (stroke (width 0) (type default))
-  )
   (wire (pts (xy 161.29 58.42) (xy 158.75 58.42))
     (stroke (width 0) (type default))
   )
-  (wire (pts (xy 33.02 114.3) (xy 33.02 111.76))
+  (wire (pts (xy 38.1 111.76) (xy 38.1 108.585))
     (stroke (width 0) (type default))
   )
@@
     (stroke (width 0) (type default))
   )
-  (wire (pts (xy 40.64 125.73) (xy 48.26 125.73))
+  (wire (pts (xy 38.1 108.585) (xy 46.99 108.585))
     (stroke (width 0) (type default))
   )
@@
     (stroke (width 0) (type default))
   )
-  (wire (pts (xy 40.64 115.57) (xy 40.64 116.84))
-    (stroke (width 0) (type default))
-  )
   (polyline (pts (xy 52.07 128.27) (xy 52.07 198.12))
     (stroke (width 0) (type default))
@@
     (stroke (width 0) (type default))
   )
-  (wire (pts (xy 48.26 111.76) (xy 46.99 111.76))
-    (stroke (width 0) (type default))
-  )
   (polyline (pts (xy 52.07 128.27) (xy 52.07 99.06))
     (stroke (width 0) (type default))
@@
   )
   (wire (pts (xy 44.45 50.8) (xy 39.37 50.8))
-    (stroke (width 0) (type default))
-  )
-  (wire (pts (xy 33.02 111.76) (xy 34.29 111.76))
     (stroke (width 0) (type default))
   )
@@
     (effects (font (size 1.27 1.27)) (justify right bottom))
   )
-  (label "BOOT1" (at 48.26 125.73 180) (fields_autoplaced)
+  (label "BOOT1" (at 46.99 108.585 180) (fields_autoplaced)
     (effects (font (size 1.27 1.27)) (justify right bottom))
   )
@@
     )
   )
-  (symbol (lib_id "power:+3.3V") (at 48.26 110.49 0) (unit 1)
-    (in_bom yes) (on_board yes) (dnp no) (fields_autoplaced)
-    (property "Reference" "#PWR023" (at 48.26 114.3 0)
-      (effects (font (size 1.27 1.27)) hide)
-    )
-    (property "Value" "+3.3V" (at 48.26 106.68 0)
-      (effects (font (size 1.27 1.27)))
-    )
-    (property "Footprint" "" (at 48.26 110.49 0)
-      (effects (font (size 1.27 1.27)) hide)
-    )
-    (property "Datasheet" "" (at 48.26 110.49 0)
-      (effects (font (size 1.27 1.27)) hide)
-    )
-    (pin "1")
-    (instances
-      (project "TER_PEDAL"
-        (path "/73ede3a3-6344-40fe-9207-10ff50d388ba/7632a94a-0691-4527-83e2-6d814eae7e64"
-          (reference "#PWR023") (unit 1)
-        )
-      )
-    )
-  )
-  (symbol (lib_id "Device:R_Small") (at 40.64 119.38 0) (unit 1)
-    (in_bom yes) (on_board yes) (dnp no) (fields_autoplaced)
-    (property "Reference" "R5" (at 43.18 118.745 0)
-      (effects (font (size 1.27 1.27)) (justify left))
-    )
-    (property "Value" "10k" (at 43.18 121.285 0)
-      (effects (font (size 1.27 1.27)) (justify left))
-    )
-    (property "Footprint" "Resistor_SMD:R_0603_1608Metric" (at 40.64 119.38 0)
-      (effects (font (size 1.27 1.27)) hide)
-    )
-    (property "Datasheet" "~" (at 40.64 119.38 0)
-      (effects (font (size 1.27 1.27)) hide)
-    )
-    (pin "1")
-    (pin "2")
-    (instances
-      (project "TER_PEDAL"
-        (path "/73ede3a3-6344-40fe-9207-10ff50d388ba/7632a94a-0691-4527-83e2-6d814eae7e64"
-          (reference "R5") (unit 1)
-        )
-      )
-    )
-  )
   (symbol (lib_id "power:+3.3VADC") (at 148.59 41.91 0) (unit 1)
     (in_bom yes) (on_board yes) (dnp no)
@@
         (path "/73ede3a3-6344-40fe-9207-10ff50d388ba/7632a94a-0691-4527-83e2-6d814eae7e64"
           (reference "C4") (unit 1)
-        )
-      )
-    )
-  )
-  (symbol (lib_id "Jumper:Jumper_3_Bridged12") (at 40.64 111.76 0) (unit 1)
-    (in_bom yes) (on_board yes) (dnp no) (fields_autoplaced)
-    (property "Reference" "JP2" (at 40.64 106.68 0)
-      (effects (font (size 1.27 1.27)))
-    )
-    (property "Value" "BOOT1" (at 40.64 109.22 0)
-      (effects (font (size 1.27 1.27)))
-    )
-    (property "Footprint" "Connector_PinHeader_2.00mm:PinHeader_1x03_P2.00mm_Vertical" (at 40.64 111.76 0)
-      (effects (font (size 1.27 1.27)) hide)
-    )
-    (property "Datasheet" "~" (at 40.64 111.76 0)
-      (effects (font (size 1.27 1.27)) hide)
-    )
-    (pin "1")
-    (pin "2")
-    (pin "3")
-    (instances
-      (project "TER_PEDAL"
-        (path "/73ede3a3-6344-40fe-9207-10ff50d388ba/7632a94a-0691-4527-83e2-6d814eae7e64"
-          (reference "JP2") (unit 1)
         )
       )
@@
     )
   )
-  (symbol (lib_id "power:GND") (at 33.02 114.3 0) (unit 1)
+  (symbol (lib_id "power:GND") (at 38.1 111.76 0) (unit 1)
     (in_bom yes) (on_board yes) (dnp no) (fields_autoplaced)
-    (property "Reference" "#PWR022" (at 33.02 120.65 0)
-      (effects (font (size 1.27 1.27)) hide)
-    )
-    (property "Value" "GND" (at 33.02 119.38 0)
-      (effects (font (size 1.27 1.27)))
-    )
-    (property "Footprint" "" (at 33.02 114.3 0)
-      (effects (font (size 1.27 1.27)) hide)
-    )
-    (property "Datasheet" "" (at 33.02 114.3 0)
-      (effects (font (size 1.27 1.27)) hide)
-    )
+    (property "Reference" "#PWR022" (at 38.1 118.11 0)
+      (effects (font (size 1.27 1.27)) hide)
+    )
+    (property "Value" "GND" (at 38.1 116.84 0)
+      (effects (font (size 1.27 1.27)))
+    )
+    (property "Footprint" "" (at 38.1 111.76 0)
+      (effects (font (size 1.27 1.27)) hide)
+    )
+    (property "Datasheet" "" (at 38.1 111.76 0)
+      (effects (font (size 1.27 1.27)) hide)
+    )

Commit message: condensador señal brake
Parts:
- renumbered C5 to C1, C1 to C2, C2 to C3, C3 to C4, C4 to C5

Commit message: Cabiado esquematico, falta layout
Parts:
- removed J1: DEBUG, Connector_PinHeader_2.00mm:PinHeader_1x04_P2.00mm_Vertical, symbol Connector:Conn_01x04_Male
- added J7: DEBUG, Connector_PinHeader_1.27mm:PinHeader_2x05_P1.27mm_Vertical, symbol Connector:Conn_ARM_JTAG_SWD_10
- added R16, R5, R8: 100k, Resistor_SMD:R_0603_1608Metric, symbol Device:R_Small
Connections:
- net +3.3V: now also J7.1 (VTref), R16.1, R5.1
- net GND: now also J7.3 (GND), J7.5 (GND), J7.9 (GNDDetect), R8.2
- net NRST: now also J7.10 (~{RESET}), R5.2
- net SWCLK: now also J7.4 (SWCLK/TCK), R8.1
- net SWDIO: now also J7.2 (SWDIO/TMS), R16.2
- new net SWO: J7.6 (SWO/TDO)
- no-connect marks 24 -> 25
