File: HARDWARE/TER_PEDAL/MICRO.kicad_sch (KiCad schematic)
At the start: 23 parts, among them J7 DEBUG, SW1 RST, SW2 BOOT0, U1 STM32F103C8Tx, Y1 8mHz

Commit message: Cambio competi resistencia 1.5k
Parts:
- renumbered C1 to C6, C5 to C7, C9 to C8
