File: HARDWARE/TER_PEDAL/TER_PEDAL.kicad_sch (KiCad schematic)
At the start: 10 parts

Commit message: Added Template to Schematics
Other:
- company: (none) -> Tecnun-eRacing
- title: (none) -> TeR_PEDAL
Changed lines of the file:
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@@
 (kicad_sch (version 20230121) (generator eeschema)
   (paper "A4")
+  (title_block
+    (title "TeR_PEDAL")
+    (date "2023-11-24")
+    (rev "V1.1.0")
+    (company "Tecnun-eRacing")
+    (comment 1 "Ozuba")
+  )
   (wire (pts (xy 54.61 168.91) (xy 49.53 168.91))
     (stroke (width 0) (type default))

Commit message: Added voltage followers to sensing, improved can circuitri, improved layout, waiting for routing
Parts:
- D3: value LED -> SYS
- D4: value LED -> IMP
- D5: value LED -> PWR
Connections:
- net DBG_LED renamed SYS
Other:
- sheet MICRO ports: added SYS; removed DBG_LED
- moved on the sheet: D5, R15
Changed lines of the file:
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@@
 	(wire
 		(pts
-			(xy 54.61 182.88) (xy 49.53 182.88)
+			(xy 54.61 177.8) (xy 49.53 177.8)
 		)
 		(stroke
@@
 	(text "POWER"
 		(exclude_from_sim no)
-		(at 64.77 184.15 0)
+		(at 64.77 179.07 0)
 		(effects
 			(font
@@
 		)
 	)
-	(label "DBG_LED"
+	(label "SYS"
 		(at 26.67 163.83 0)
 		(fields_autoplaced yes)
@@
 		)
 	)
-	(label "DBG_LED"
+	(label "SYS"
 		(at 161.29 96.52 180)
 		(fields_autoplaced yes)
@@
 	(symbol
 		(lib_id "power:GND")
-		(at 54.61 182.88 90)
+		(at 54.61 177.8 90)
 		(mirror x)
 		(unit 1)
@@
 		(fields_autoplaced yes)
 		(property "Reference" "#PWR045"
-			(at 60.96 182.88 0)
+			(at 60.96 177.8 0)
 			(effects
 				(font
@@
 		)
 		(property "Value" "GND"
-			(at 58.42 183.515 90)
+			(at 58.42 178.435 90)
 			(effects
 				(font
@@
 		)
 		(property "Footprint" ""
-			(at 54.61 182.88 0)
+			(at 54.61 177.8 0)
 			(effects
 				(font
@@
 		)
 		(property "Datasheet" ""
-			(at 54.61 182.88 0)
+			(at 54.61 177.8 0)
 			(effects
 				(font
@@
 		)
 		(property "Description" ""
-			(at 54.61 182.88 0)
+			(at 54.61 177.8 0)
 			(effects
 				(font
@@
 			)
 		)
-		(property "Value" "LED"
+		(property "Value" "SYS"
 			(at 45.72 161.29 0)
 			(effects
@@
 	(symbol
 		(lib_id "Device:LED")
-		(at 45.72 182.88 0)
+		(at 45.72 177.8 0)
 		(mirror y)
 		(unit 1)
@@
 		(dnp no)
 		(property "Reference" "D5"
-			(at 46.99 186.69 0)
-			(effects
-				(font
-					(size 1.27 1.27)
-				)
-			)
-		)
-		(property "Value" "LED"
-			(at 45.72 180.34 0)
+			(at 46.99 181.61 0)
+			(effects
+				(font
+					(size 1.27 1.27)
+				)
+			)
+		)
+		(property "Value" "PWR"
+			(at 45.72 175.26 0)
 			(effects
 				(font
@@
 		)
 		(property "Footprint" "LED_SMD:LED_0603_1608Metric"
-			(at 45.72 182.88 0)
+			(at 45.72 177.8 0)
 			(effects
 				(font
@@
 		)
 		(property "Datasheet" "~"
-			(at 45.72 182.88 0)
+			(at 45.72 177.8 0)
 			(effects
 				(font
@@
 		)
 		(property "Description" ""
-			(at 45.72 182.88 0)
+			(at 45.72 177.8 0)
 			(effects
 				(font
@@
 			)
 		)
-		(property "Value" "LED"
+		(property "Value" "IMP"
 			(at 45.72 166.37 0)
 			(effects
@@
 	(symbol
 		(lib_id "power:+3.3V")
-		(at 34.29 182.88 90)
+		(at 34.29 177.8 90)
 		(unit 1)
 		(exclude_from_sim no)
@@
 		(fields_autoplaced yes)
 		(property "Reference" "#PWR046"
-			(at 38.1 182.88 0)
+			(at 38.1 177.8 0)
 			(effects
 				(font
@@
 		)
 		(property "Value" "+3.3V"
-			(at 30.48 183.515 90)
+			(at 30.48 178.435 90)
 			(effects
 				(font
@@
 		)
 		(property "Footprint" ""
-			(at 34.29 182.88 0)
+			(at 34.29 177.8 0)
 			(effects
 				(font
@@
 		)
 		(property "Datasheet" ""
-			(at 34.29 182.88 0)
+			(at 34.29 177.8 0)
 			(effects
 				(font
@@
 		)
 		(property "Description" ""
-			(at 34.29 182.88 0)
+			(at 34.29 177.8 0)
 			(effects
 				(font
@@
 	(symbol
 		(lib_id "Device:R")
-		(at 38.1 182.88 270)
+		(at 38.1 177.8 270)
 		(mirror x)
 		(unit 1)
@@
 		(dnp no)
 		(property "Reference" "R15"
-			(at 38.1 185.42 90)
+			(at 38.1 180.34 90)
 			(effects
 				(font
@@
 		)
 		(property "Value" "120R"
-			(at 38.1 180.34 90)
+			(at 38.1 175.26 90)
 			(effects
 				(font
@@
 		)
 		(property "Footprint" "Capacitor_SMD:C_0402_1005Metric"
-			(at 38.1 184.658 90)
+			(at 38.1 179.578 90)
 			(effects
 				(font
@@
 		)
 		(property "Datasheet" "~"
-			(at 38.1 182.88 0)
+			(at 38.1 177.8 0)
 			(effects
 				(font
@@
 		)
 		(property "Description" ""
-			(at 38.1 182.88 0)
+			(at 38.1 177.8 0)
 			(effects
 				(font
@@
 			)
 		)
-		(pin "DBG_LED" input
-			(at 149.86 96.52 0)
-			(effects
-				(font
-					(size 1.27 1.27)
-				)
-				(justify right)
-			)
-		)
 		(pin "APPS_2_ADC" input
 			(at 121.92 73.66 180)
@@
 			)
 		)
+		(pin "SYS" input
+			(at 149.86 96.52 0)
+			(effects
+				(font
+					(size 1.27 1.27)
+				)
+				(justify right)
+			)
+		)
 		(instances
 			(project "TER_PEDAL"
@@
 	(sheet
 		(at 171.45 36.83)
-		(size 31.75 21.59)
+		(size 31.75 19.05)
 		(fields_autoplaced yes)
 		(stroke
@@
 		)
 		(property "Sheetfile" "CAN.kicad_sch"
-			(at 171.45 59.0046 0)
-			(effects
-				(font
+			(at 171.45 56.4646 0)
+			(effects
+				(font

Commit message: Añadiendo eeprom (no terminado)
Other:
- added sheet EEPROM (EEPROM.kicad_sch)
- sheet MICRO ports: added SCL, SDA; removed none
Changed lines of the file:
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@@
+	(wire
+		(pts
+			(xy 149.86 73.025) (xy 163.195 73.025)
+		)
+		(stroke
+			(width 0)
+			(type default)
+		)
+	)
 	(wire
 		(pts
@@
 		(pts
 			(xy 107.95 73.66) (xy 121.92 73.66)
+		)
+		(stroke
+			(width 0)
+			(type default)
+		)
+	)
+	(wire
+		(pts
+			(xy 149.86 76.835) (xy 163.195 76.835)
 		)
 		(stroke
@@
 	)
 	(sheet
+		(at 163.195 69.596)
+		(size 21.336 14.732)
+		(fields_autoplaced yes)
+		(stroke
+			(width 0.1524)
+			(type solid)
+		)
+		(fill
+			(color 0 0 0 0.0000)
+		)
+		(property "Sheetname" "EEPROM"
+			(at 163.195 68.8844 0)
+			(effects
+				(font
+					(size 1.27 1.27)
+				)
+				(justify left bottom)
+			)
+		)
+		(property "Sheetfile" "EEPROM.kicad_sch"
+			(at 163.195 84.9126 0)
+			(effects
+				(font
+					(size 1.27 1.27)
+				)
+				(justify left top)
+			)
+		)
+		(pin "SDA" input
+			(at 163.195 73.025 180)
+			(effects
+				(font
+					(size 1.27 1.27)
+				)
+				(justify left)
+			)
+		)
+		(pin "SCL" input
+			(at 163.195 76.835 180)
+			(effects
+				(font
+					(size 1.27 1.27)
+				)
+				(justify left)
+			)
+		)
+		(instances
+			(project "TER_PEDAL"
+				(path "/73ede3a3-6344-40fe-9207-10ff50d388ba"
+					(page "7")
+				)
+			)
+		)
+	)
+	(sheet
 		(at 223.52 38.1)
 		(size 26.67 19.05)
@@
 			(effects
 				(font
+					(size 1.27 1.27)
+				)
+				(justify right)
+			)
+		)
+		(pin "SDA" input
+			(at 149.86 73.025 0)
+			(effects
+				(font
+					(size 1.27 1.27)
+				)
+				(justify right)
+			)
+		)
+		(pin "SCL" input
+			(at 149.86 76.835 0)
+			(effects
+				(font
