File: HARDWARE/TER_PEDAL/_autosave-TER_PEDAL.kicad_pcb (KiCad board)
At the start: 4 copper layers, 78.6 x 34.5 mm, 81 parts, among them J1 APPS_2, J2 APPS_1, J3 RJ45_Shielded, J4 APPS_1, J5 BPPS_1, J7 DEBUG, SW1 RST, SW2 BOOT0, U1 STM32F103C8Tx, U2 TSR_1-2450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

Commit message: EEPROM añadida
Other:
- board text removed: "falta pull ups"
Changed lines of the file:
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@@
-		)
-	)
-	(gr_text "falta pull ups"
-		(at 133.32 74.89 0)
-		(layer "Cmts.User")
-		(effects
-			(font
-				(size 1.5 1.5)
-				(thickness 0.3)
-				(bold yes)
-			)
-			(justify left bottom)
 		)
 	)
