File: HARDWARE/TER_PEDAL/SENSORS.kicad_sch (KiCad schematic)
At the start: 25 parts, among them J1 APPS_2, J2 APPS_1, J4 APPS_1, J5 BPPS_1, U4 LM321, U6 LM321, U7 LM321, U8 LM321

Commit message: Cambio competi resistencia 1.5k
Parts:
- R2: value 0R -> 1.5k
